File: luxometro_16F1709.sch (EAGLE design)
At the start: 12 parts, among them IC1 7805, X1 22-23-2021

Commit message: Esquema
Cambios en esquema.
Parts:
- added C4: 18p, rcl:C-EU050-024X044
Connections:
- removed net N$10: JP4.1, R1.2, U$1.RC4/C2OUT/PH2
- new net N$12: C4.2, JP4.1, R1.2, U$1.RC4/C2OUT/PH2
- net AGND: now also JP3.1; no longer JP3.2
- net N$7: now also C4.1, JP3.2; no longer JP3.1
Other:
- note added: "Luxometro"
- moved on the sheet: JP3
